Commit message: update the urdf models

File: urdf_models/model_l0kg-r0kg.urdf (robot description, URDF)
Before this commit: robot iCub, 53 links, 52 joints
Links:
- link l_elbow_1: mass 0.347 -> 0.712463
- link r_elbow_1: mass 0.347 -> 0.750299

File: urdf_models/model_l0kg-r10kg.urdf (robot description, URDF)
Before this commit: robot iCub, 57 links, 56 joints
Links:
- removed link r_bolt_in
- link l_elbow_1: mass 0.347 -> 0.712463
- link r_elbow_1: mass 0.347 -> 0.750299
Joints:
- removed joint r_weight_stacked0
- joint r_weight_fixed: child r_bolt_in -> r_weight_5

File: urdf_models/model_l0kg-r7kg.urdf (robot description, URDF)
Before this commit: robot iCub, 57 links, 56 joints
Links:
- removed link r_bolt_in
- link l_elbow_1: mass 0.347 -> 0.712463
- link r_elbow_1: mass 0.347 -> 0.750299
Joints:
- removed joint r_weight_stacked0
- joint r_weight_fixed: child r_bolt_in -> r_weight_5

File: urdf_models/model_l2kg-r2kg.urdf (robot description, URDF)
Before this commit: robot iCub, 59 links, 58 joints
Links:
- removed link l_bolt_in
- removed link r_bolt_in
- link l_elbow_1: mass 0.347 -> 0.712463
- link r_elbow_1: mass 0.347 -> 0.750299
Joints:
- removed joint l_weight_stacked00
- removed joint r_weight_stacked00
- joint l_weight_fixed: child l_bolt_in -> l_weight_2a
- joint r_weight_fixed: child r_bolt_in -> r_weight_2a

File: urdf_models/model_l4kg-r4kg.urdf (robot description, URDF)
Before this commit: robot iCub, 61 links, 60 joints
Links:
- removed link l_bolt_in
- removed link r_bolt_in
- link l_elbow_1: mass 0.347 -> 0.712463
- link r_elbow_1: mass 0.347 -> 0.750299
Joints:
- removed joint l_weight_stacked00
- removed joint r_weight_stacked00
- joint l_weight_fixed: child l_bolt_in -> l_weight_2a
- joint r_weight_fixed: child r_bolt_in -> r_weight_2a

File: urdf_models/model_l5kg-r0kg.urdf (robot description, URDF)
Before this commit: robot iCub, 56 links, 55 joints
Links:
- removed link l_bolt_in
- link l_elbow_1: mass 0.347 -> 0.712463
- link r_elbow_1: mass 0.347 -> 0.750299
Joints:
- removed joint l_weight_stacked0
- joint l_weight_fixed: child l_bolt_in -> l_weight_5

File: urdf_models/model_l5kg-r5kg.urdf (robot description, URDF)
Before this commit: robot iCub, 59 links, 58 joints
Links:
- removed link l_bolt_in
- removed link r_bolt_in
- link l_elbow_1: mass 0.347 -> 0.712463
- link r_elbow_1: mass 0.347 -> 0.750299
Joints:
- removed joint l_weight_stacked0
- removed joint r_weight_stacked0
- joint l_weight_fixed: child l_bolt_in -> l_weight_5
- joint r_weight_fixed: child r_bolt_in -> r_weight_5
